Commit message: chore: update bazel configuration and build files

File: ros2/test/xacro/sample2.xacro (robot description, xacro)
@@ -1,4 +1,4 @@
 <xml xmlns:xacro="http://www.ros.org/wiki/xacro">
-  <xacro:include filename="$(cwd)/ros2/test/xacro/sample1.xacro" />
+  <xacro:include filename="sample1.xacro" />
   <xacro:macro name="m" params="foo"><a foo="${foo}"/></xacro:macro>
   <xacro:m foo="1 ${foo}"/>

File: ros2/test/xacro/test_with_params.xacro (robot description, xacro)
@@ -1,4 +1,4 @@
 <xml xmlns:xacro="http://www.ros.org/wiki/xacro">
-  <xacro:property name="yaml_file" value="$(cwd)/ros2/test/xacro/params.yaml" />
+  <xacro:property name="yaml_file" value="params.yaml" />
   <xacro:property name="props" value="${load_yaml(yaml_file)}"/>
   <xacro:property name="val1" value="${props['foo']}" />
