Commit message: Update ros2_diagnostics, xacro, urdf, orocos_kdl to versions matching Jazzy
- ros2_diagnostics: bump to release tag 4.5.7; diagnostic_updater now ships
  its implementation in a separate .cpp instead of being header-only, so
  add it to the cc_library srcs.
- ros2_xacro: bump to 2.1.1, matching Jazzy's rosdistro pin. Fix a test
  fixture using the now-deprecated load_yaml() free function in favor of
  xacro.load_yaml().
- ros2_urdf: bump to 2.10.1, matching Jazzy's rosdistro pin.
- orocos_kdl: bump to the commit pinned by orocos_kdl_vendor's 0.5.2 tag
  (Jazzy's release), replacing the older commit pinned via 0.2.5.

Verified via bazel build/test of the affected targets (diagnostics,
xacro, geometry2, urdf, robot_state_publisher, kdl_parser tests/builds).

Co-Authored-By: Claude Sonnet 5 <noreply@anthropic.com>

File: ros2/test/xacro/test_with_params.xacro (robot description, xacro)
@@ -1,5 +1,5 @@
 <xml xmlns:xacro="http://www.ros.org/wiki/xacro">
   <xacro:property name="yaml_file" value="$(cwd)/ros2/test/xacro/params.yaml" />
-  <xacro:property name="props" value="${load_yaml(yaml_file)}"/>
+  <xacro:property name="props" value="${xacro.load_yaml(yaml_file)}"/>
   <xacro:property name="val1" value="${props['foo']}" />
   <a foo="${props['foo']}"/>
